File: arc-dvi-vidc-brds.kicad_sch (KiCad schematic)
At the start: 25 parts, among them IC1 SN74ALVC164245, IC2 SN74ALVC164245, IC3 SN74ALVC164245, J1 Connector_50pin_FFC, U1 MIC5219 3.3V

Commit message: Pretty much finished
Not DRC'd though, FIXME.  Routed, with dimensions measured from
A3000/FDD spacing etc.  Includes extra 80mm holes to mount the
podule board under FDD too.
Parts:
- added R1, R2: 4K7, Resistor_SMD:R_0603_1608Metric, symbol Device:R_Small
Connections:
- net +3V3: now also R1.1
- net CKIN: now also IC3.14 (2B2); no longer IC3.20 (2B6)
- net FLYBK: now also IC3.16 (2B3); no longer IC3.17 (2B4)
- net GND: now also R2.2
- net NHS: now also IC3.22 (2B7); no longer IC3.14 (2B2)
- net NSNDRQ: now also IC3.17 (2B4); no longer IC3.16 (2B3)
- net NVCS: now also IC3.20 (2B6); no longer IC3.13 (2B1)
- net NVIDW: now also IC3.23 (2B8); no longer IC3.12 (1B8)
- net SNDAK: now also IC3.12 (1B8); no longer IC3.22 (2B7)
- net VIDAK: now also IC3.13 (2B1); no longer IC3.23 (2B8)
- net ID_DET: now reaches J1.49
- net ID_DET: now also R1.2, R2.1
Changed lines of the file:
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@@
   (junction (at 289.56 330.2) (diameter 0) (color 0 0 0 0)
   )
+  (junction (at 464.82 346.71) (diameter 0) (color 0 0 0 0)
+  )
   (junction (at 289.56 322.58) (diameter 0) (color 0 0 0 0)
   )
@@
     (stroke (width 0) (type default) (color 0 0 0 0))
   )
+  (wire (pts (xy 464.82 345.44) (xy 464.82 346.71))
+    (stroke (width 0) (type default) (color 0 0 0 0))
+  )
   (wire (pts (xy 99.06 189.23) (xy 130.81 189.23))
     (stroke (width 0) (type default) (color 0 0 0 0))
@@
     (stroke (width 0) (type default) (color 0 0 0 0))
   )
+  (wire (pts (xy 464.82 353.06) (xy 464.82 355.6))
+    (stroke (width 0) (type default) (color 0 0 0 0))
+  )
   (wire (pts (xy 353.06 129.54) (xy 433.07 129.54))
     (stroke (width 0) (type default) (color 0 0 0 0))
@@
     (stroke (width 0) (type default) (color 0 0 0 0))
   )
+  (wire (pts (xy 458.47 304.8) (xy 471.17 304.8))
+    (stroke (width 0) (type default) (color 0 0 0 0))
+  )
   (wire (pts (xy 455.93 195.58) (xy 471.17 195.58))
     (stroke (width 0) (type default) (color 0 0 0 0))
@@
     (stroke (width 0) (type default) (color 0 0 0 0))
   )
+  (wire (pts (xy 464.82 337.82) (xy 464.82 340.36))
+    (stroke (width 0) (type default) (color 0 0 0 0))
+  )
   (wire (pts (xy 403.86 231.14) (xy 471.17 231.14))
     (stroke (width 0) (type default) (color 0 0 0 0))
@@
     (stroke (width 0) (type default) (color 0 0 0 0))
   )
+  (wire (pts (xy 464.82 346.71) (xy 478.79 346.71))
+    (stroke (width 0) (type default) (color 0 0 0 0))
+  )
   (wire (pts (xy 353.06 210.82) (xy 375.92 210.82))
     (stroke (width 0) (type default) (color 0 0 0 0))
@@
     (stroke (width 0) (type default) (color 0 0 0 0))
   )
+  (wire (pts (xy 464.82 346.71) (xy 464.82 347.98))
+    (stroke (width 0) (type default) (color 0 0 0 0))
+  )
   (wire (pts (xy 99.06 173.99) (xy 130.81 173.99))
     (stroke (width 0) (type default) (color 0 0 0 0))
@@
     (effects (font (size 1.2446 1.2446)) (justify left bottom))
   )
-  (label "NVIDW" (at 302.26 299.72 0)
+  (label "NVIDW" (at 302.26 327.66 0)
     (effects (font (size 1.2446 1.2446)) (justify left bottom))
   )
@@
     (effects (font (size 1.2446 1.2446)) (justify left bottom))
   )
-  (label "FLYBK" (at 302.26 312.42 0)
+  (label "FLYBK" (at 302.26 309.88 0)
     (effects (font (size 1.2446 1.2446)) (justify left bottom))
   )
@@
     (effects (font (size 1.2446 1.2446)) (justify left bottom))
   )
-  (label "NSNDRQ" (at 302.26 309.88 0)
+  (label "NSNDRQ" (at 302.26 312.42 0)
     (effects (font (size 1.2446 1.2446)) (justify left bottom))
   )
+  (label "ID_DET" (at 458.47 304.8 0)
+    (effects (font (size 1.27 1.27)) (justify left bottom))
+  )
   (label "D6" (at 302.26 157.48 0)
     (effects (font (size 1.2446 1.2446)) (justify left bottom))
@@
     (effects (font (size 1.2446 1.2446)) (justify left bottom))
   )
-  (label "NHS" (at 302.26 304.8 0)
+  (label "NHS" (at 302.26 325.12 0)
     (effects (font (size 1.2446 1.2446)) (justify left bottom))
   )
@@
     (effects (font (size 1.2446 1.2446)) (justify left bottom))
   )
-  (label "SNDAK" (at 302.26 325.12 0)
+  (label "SNDAK" (at 302.26 299.72 0)
     (effects (font (size 1.2446 1.2446)) (justify left bottom))
   )
@@
     (effects (font (size 1.2446 1.2446)) (justify left bottom))
   )
+  (label "ID_DET" (at 478.79 346.71 0)
+    (effects (font (size 1.27 1.27)) (justify left bottom))
+  )
   (label "D1" (at 130.81 212.09 0)
     (effects (font (size 1.2446 1.2446)) (justify left bottom))
@@
     (effects (font (size 1.2446 1.2446)) (justify left bottom))
   )
-  (label "VIDAK" (at 302.26 327.66 0)
+  (label "VIDAK" (at 302.26 302.26 0)
     (effects (font (size 1.2446 1.2446)) (justify left bottom))
   )
@@
     (effects (font (size 1.2446 1.2446)) (justify left bottom))
   )
-  (label "CKIN" (at 302.26 320.04 0)
+  (label "CKIN" (at 302.26 304.8 0)
     (effects (font (size 1.2446 1.2446)) (justify left bottom))
   )
@@
     (effects (font (size 1.2446 1.2446)) (justify left bottom))
   )
-  (label "NVCS" (at 302.26 302.26 0)
+  (label "NVCS" (at 302.26 320.04 0)
     (effects (font (size 1.2446 1.2446)) (justify left bottom))
   )
@@
     (pin "5")
   )
+  (symbol (lib_id "Device:R_Small") (at 464.82 342.9 0) (unit 1)
+    (in_bom no) (on_board yes) (fields_autoplaced)
+    (property "Reference" "R1" (id 0) (at 467.36 341.6299 0)
+      (effects (font (size 1.27 1.27)) (justify left))
+    )
+    (property "Value" "4K7" (id 1) (at 467.36 344.1699 0)
+      (effects (font (size 1.27 1.27)) (justify left))
+    )
+    (property "Footprint" "Resistor_SMD:R_0603_1608Metric" (id 2) (at 464.82 342.9 0)
+      (effects (font (size 1.27 1.27)) hide)
+    )
+    (property "Datasheet" "~" (id 3) (at 464.82 342.9 0)
+      (effects (font (size 1.27 1.27)) hide)
+    )
+    (pin "1")
+    (pin "2")
+  )
   (symbol (lib_id "arc-dvi-vidc-brds-eagle-import:4R-NCAY16") (at 347.98 210.82 0) (unit 4)
     (in_bom yes) (on_board yes)
@@
     (pin "1")
   )
+  (symbol (lib_id "arc-dvi-vidc-brds-eagle-import:+3V3") (at 464.82 335.28 0) (unit 1)
+    (in_bom yes) (on_board yes)
+    (property "Reference" "#+3V0101" (id 0) (at 464.82 335.28 0)
+      (effects (font (size 1.27 1.27)) hide)
+    )
+    (property "Value" "+3V3" (id 1) (at 462.28 340.36 90)
+      (effects (font (size 1.778 1.5113)) (justify left bottom))
+    )
+    (property "Footprint" "arc-dvi-vidc-brds:" (id 2) (at 464.82 335.28 0)
+      (effects (font (size 1.27 1.27)) hide)
+    )
+    (property "Datasheet" "" (id 3) (at 464.82 335.28 0)
+      (effects (font (size 1.27 1.27)) hide)
+    )
+    (pin "1")
+  )
   (symbol (lib_id "arc-dvi-vidc-brds-eagle-import:4R-NCAY16") (at 347.98 177.8 0) (unit 3)
     (in_bom yes) (on_board yes)
@@
     (pin "5")
   )
+  (symbol (lib_id "Device:R_Small") (at 464.82 350.52 0) (unit 1)
+    (in_bom yes) (on_board yes) (fields_autoplaced)
+    (property "Reference" "R2" (id 0) (at 467.36 349.2499 0)
+      (effects (font (size 1.27 1.27)) (justify left))
+    )
+    (property "Value" "4K7" (id 1) (at 467.36 351.7899 0)
+      (effects (font (size 1.27 1.27)) (justify left))
+    )
+    (property "Footprint" "Resistor_SMD:R_0603_1608Metric" (id 2) (at 464.82 350.52 0)
+      (effects (font (size 1.27 1.27)) hide)
+    )
+    (property "Datasheet" "~" (id 3) (at 464.82 350.52 0)
+      (effects (font (size 1.27 1.27)) hide)
+    )
+    (pin "1")
+    (pin "2")
+  )
   (symbol (lib_id "arc-dvi-vidc-brds-eagle-import:4R-NCAY16") (at 347.98 302.26 0) (unit 1)
     (in_bom yes) (on_board yes)
@@
     (pin "5")
   )
+  (symbol (lib_id "arc-dvi-vidc-brds-eagle-import:GND") (at 464.82 358.14 0) (unit 1)
+    (in_bom yes) (on_board yes)
+    (property "Reference" "#GND0102" (id 0) (at 464.82 358.14 0)
+      (effects (font (size 1.27 1.27)) hide)
+    )
+    (property "Value" "GND" (id 1) (at 462.28 360.68 0)
+      (effects (font (size 1.778 1.5113)) (justify left bottom))
+    )
+    (property "Footprint" "arc-dvi-vidc-brds:" (id 2) (at 464.82 358.14 0)
+      (effects (font (size 1.27 1.27)) hide)
+    )
+    (property "Datasheet" "" (id 3) (at 464.82 358.14 0)
+      (effects (font (size 1.27 1.27)) hide)
+    )
+    (pin "1")
+  )
   (symbol (lib_id "arc-dvi-vidc-brds-eagle-import:4R-NCAY16") (at 347.98 154.94 0) (unit 1)
     (in_bom yes) (on_board yes)
@@
       (reference "#+3V03") (unit 1) (value "+3V3") (footprint "arc-dvi-vidc-brds:")
     )
+    (path "/6d9e6ee3-5a8f-4273-863f-7b84416aa188"
+      (reference "#+3V0101") (unit 1) (value "+3V3") (footprint "arc-dvi-vidc-brds:")
+    )
     (path "/c3c8b42e-f0ce-4680-a161-761383c7f31f"
       (reference "#FRAME1") (unit 2) (value "FRAME_C_L") (footprint "arc-dvi-vidc-brds:")
@@
       (reference "#GND0101") (unit 1) (value "GND") (footprint "arc-dvi-vidc-brds:")
     )
+    (path "/dded0e57-6975-4084-9d40-5ce5c7f322a4"
+      (reference "#GND0102") (unit 1) (value "GND") (footprint "arc-dvi-vidc-brds:")
+    )
     (path "/76e3d594-f7b1-4132-a636-2dacb680f822"
       (reference "#P+02") (unit 1) (value "+5V") (footprint "arc-dvi-vidc-brds:")
@@
       (reference "J1") (unit 1) (value "Connector_50pin_FFC") (footprint "Connector_FFC-FPC:Hirose_FH12-50S-0.5SH_1x50-1MP_P0.50mm_Horizontal")
     )
+    (path "/0cfa998a-511c-46d0-ba84-3cf02bc7a48c"
+      (reference "R1") (unit 1) (value "4K7") (footprint "Resistor_SMD:R_0603_1608Metric")
+    )
+    (path "/d3bd2271-b989-47f5-8096-2f4190a6ce3a"
+      (reference "R2") (unit 1) (value "4K7") (footprint "Resistor_SMD:R_0603_1608Metric")
+    )
     (path "/8f72ca2d-7d88-4126-97f0-ea0cb26cd904"

Commit message: Add README, licence
Other:
- note added: "24 April 2023"
- note added: "Copyright 2021-2023 Matt Evans CC BY-NC-SA 3.0"
- note removed: "(c) 2021 Matt Evans"
- note removed: "22 Oct 2021"
Changed lines of the file:
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@@
     (stroke (width 0) (type default) (color 0 0 0 0))
   )
-  (text "VIDC interposer board" (at 474.98 419.1 180)
+  (text "VIDC interposer board" (at 478.79 430.53 180)
     (effects (font (size 1.778 1.5113)) (justify left bottom))
   )
-  (text "(For A3000/soldered VIDC)" (at 510.54 419.1 180)
+  (text "(For A3000/soldered VIDC)" (at 501.65 435.61 180)
     (effects (font (size 1.778 1.5113)) (justify left bottom))
   )
@@
     (effects (font (size 5 5)) (justify left bottom))
   )
-  (text "22 Oct 2021" (at 474.98 424.18 180)
+  (text "24 April 2023" (at 478.79 435.61 180)
     (effects (font (size 1.778 1.5113)) (justify left bottom))
   )
@@
     (effects (font (size 1.778 1.5113)) (justify left bottom))
   )
-  (text "(c) 2021 Matt Evans" (at 535.94 424.18 180)
+  (text "Copyright 2021-2023 Matt Evans\n\nCC BY-NC-SA 3.0" (at 537.21 435.61 180)
     (effects (font (size 1.778 1.5113)) (justify left bottom))
   )
-  (text "v2" (at 561.34 441.96 180)
+  (text "v2" (at 570.23 454.66 180)
     (effects (font (size 1.778 1.5113)) (justify left bottom))
   )
@@
     (pin "5")
   )
-  (symbol (lib_id "arc-dvi-vidc-brds-eagle-import:FRAME_C_L") (at 469.9 449.58 0) (unit 2)
-    (in_bom no) (on_board no)
-    (property "Reference" "#FRAME1" (id 0) (at 469.9 449.58 0)
-      (effects (font (size 1.27 1.27)) hide)
-    )
-    (property "Value" "FRAME_C_L" (id 1) (at 469.9 449.58 0)
-      (effects (font (size 1.27 1.27)) hide)
-    )
-    (property "Footprint" "arc-dvi-vidc-brds:" (id 2) (at 469.9 449.58 0)
-      (effects (font (size 1.27 1.27)) hide)
-    )
-    (property "Datasheet" "" (id 3) (at 469.9 449.58 0)
-      (effects (font (size 1.27 1.27)) hide)
-    )
-  )
   (symbol (lib_id "arc-dvi-vidc-brds-eagle-import:4R-NCAY16") (at 347.98 137.16 0) (unit 4)
     (in_bom yes) (on_board yes)
@@
       (reference "#+3V0101") (unit 1) (value "+3V3") (footprint "arc-dvi-vidc-brds:")
     )
-    (path "/c3c8b42e-f0ce-4680-a161-761383c7f31f"
-      (reference "#FRAME1") (unit 2) (value "FRAME_C_L") (footprint "arc-dvi-vidc-brds:")
-    )
     (path "/ee5371cd-a0e6-47b9-bc43-7227b6533f0d"
